Commit message: Changed parameters to match other scripts

File: rotors_description/urdf/voliro.xacro (robot description, xacro)
@@ -35,8 +35,11 @@
     <xacro:property name="rotor_offset_top" value="0.060"/>    <!-- [m] -->
     <xacro:property name="radius_rotor" value="0.1143"/>    <!-- [m] -->
-    <xacro:property name="motor_constant" value="${8.54858e-06}"/>    <!-- [kg m/s^2] -->
-    <xacro:property name="motor_constant_lower" value="${8.54858e-06}"/>    <!-- [kg m/s^2] -->
+    <!-- <xacro:property name="motor_constant" value="${8.54858e-06}"/>    -->
+    <!-- <xacro:property name="motor_constant_lower" value="${8.54858e-06}"/>    -->
+    <xacro:property name="motor_constant" value="${7.2e-06}"/>    <!-- [kg m/s^2] -->
+    <xacro:property name="motor_constant_lower" value="${7.2e-06}"/>    <!-- [kg m/s^2] -->
     <xacro:property name="moment_constant" value="0.015"/>    <!-- [m] -->
-    <xacro:property name="moment_constant_lower" value="0.005"/>    <!-- [m] -->
+    <!-- <xacro:property name="moment_constant_lower" value="0.005"/>     -->
+    <xacro:property name="moment_constant_lower" value="0.015"/>    <!-- [m] -->
     <xacro:property name="time_constant_up" value="0.0125"/>    <!-- [s] -->
     <xacro:property name="time_constant_down" value="0.025"/>    <!-- [s] -->
@@ -56,5 +59,6 @@
     <!-- Body Interia / CoM Offset -->
     <xacro:property name="body_inertia_origin">
-      <origin xyz="0 0 -0.05" />
+      <!-- <origin xyz="0 0 -0.05" /> -->
+      <origin xyz="0 0 0.0" />
     </xacro:property>
     <!-- Rotor unit inertia without the propellor. -->

File: rotors_description/urdf/voliro_base.xacro (robot description, xacro)
@@ -24,4 +24,22 @@
   <!-- Mount an ADIS16448 IMU. -->
   <xacro:default_imu namespace="${namespace}" parent_link="${namespace}/base_link"/>
+  <!-- Mount an ADIS16448 IMU. -->
+    <!-- <xacro:imu_plugin_macro
+      namespace="${namespace}"
+      imu_suffix=""
+      parent_link="${namespace}/base_link"
+      imu_topic="/imu"
+      mass_imu_sensor="0.015"
+      gyroscope_noise_density="0.0003394"
+      gyroscope_random_walk="0.000038785"
+      gyroscope_bias_correlation_time="1000.0"
+      gyroscope_turn_on_bias_sigma="0.0087"
+      accelerometer_noise_density="0.004"
+      accelerometer_random_walk="0.006"
+      accelerometer_bias_correlation_time="300.0"
+      accelerometer_turn_on_bias_sigma="0.1960">
+      <inertia ixx="0.00001" ixy="0.0" ixz="0.0" iyy="0.00001" iyz="0.0" izz="0.00001" />
+      <origin xyz="0 0 0" rpy="0 0 0" />
+    </xacro:imu_plugin_macro> -->
   <xacro:if value="$(arg enable_ground_truth)">
       <xacro:ground_truth_imu_and_odometry
